File: control_board/lights.kicad_pcb (KiCad board)
At the start: 2 copper layers, 20 parts, among them J1 CONN_01X08, J2 CONN_01X02, U1 PCA9685PW, U2 MBI1801, U3 MBI1801, U4 MBI1801, U5 MBI1801

Commit message: control_brd: update PCB design
Parts:
- J2: footprint Connectors:AK300-2 -> Connectors:bornier2
