File: control_board/ctrl_board.kicad_pcb (KiCad board)
At the start: 2 copper layers, 130 x 130 mm, 37 parts, among them J1 CONN_01X04, J2 CONN_01X02, J3 CONN_01X04, J4 CONN_01X04, J5 CONN_01X04, J6 CONN_01X04, J7 CONN_01X04, J8 CONN_01X04, U1 PCA9685PW, U2 MBI1801, U3 MBI1801, U4 MBI1801, U5 MBI1801, U6 MBI1801, U7 MBI1801

Commit message: ctrl_board: [wip] place and route
Parts:
- moved G2 1.00 mm to (0.00, -57.0)
Other:
- board text added: "rev. 1.0 github: wojtekbe/rgbir-lights"
Changed lines of the file:
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@@
     (area -69.23219 -65.5 73.032191 70.236952)
     (thickness 1.6)
-    (drawings 480)
+    (drawings 481)
     (tracks 377)
     (zones 0)
@@
   (layers
     (0 F.Cu signal)
-    (31 B.Cu signal hide)
+    (31 B.Cu signal)
     (32 B.Adhes user)
     (33 F.Adhes user)
@@
   )
   (setup
-    (last_trace_width 0.3048)
+    (last_trace_width 0.3047)
     (user_trace_width 0.3048)
     (user_trace_width 0.6095)
@@
     (pad_to_mask_clearance 0.2)
     (aux_axis_origin -471.805 113.03)
-    (visible_elements FFFFAF7F)
+    (visible_elements FFFFBF7F)
     (pcbplotparams
       (layerselection 0x00030_ffffffff)
@@
       (effects (font (thickness 0.15)))
     )
-    (pad 1 np_thru_hole circle (at -7.5 5 300) (size 3.1 3.1) (drill 3.1) (layers *.Cu *.Mask))
-    (pad 2 np_thru_hole circle (at 7.5 5 300) (size 3.1 3.1) (drill 3.1) (layers *.Cu *.Mask))
-    (pad 3 np_thru_hole circle (at 0 -5 300) (size 3.1 3.1) (drill 3.1) (layers *.Cu *.Mask))
+    (pad 3 np_thru_hole circle (at 0 -5 300) (size 3 3) (drill 3) (layers *.Cu *.Mask))
+    (pad 2 np_thru_hole circle (at 7.5 5 300) (size 3 3) (drill 3) (layers *.Cu *.Mask))
+    (pad 1 np_thru_hole circle (at -7.5 5 300) (size 3 3) (drill 3) (layers *.Cu *.Mask))
   )
   (module generated:Mounting_holes (layer F.Cu)
@@
       (effects (font (thickness 0.15)))
     )
-    (pad 3 np_thru_hole circle (at 0 -5 60) (size 3.1 3.1) (drill 3.1) (layers *.Cu *.Mask))
-    (pad 2 np_thru_hole circle (at 7.5 5 60) (size 3.1 3.1) (drill 3.1) (layers *.Cu *.Mask))
-    (pad 1 np_thru_hole circle (at -7.5 5 60) (size 3.1 3.1) (drill 3.1) (layers *.Cu *.Mask))
+    (pad 3 np_thru_hole circle (at 0 -5 60) (size 3 3) (drill 3) (layers *.Cu *.Mask))
+    (pad 2 np_thru_hole circle (at 7.5 5 60) (size 3 3) (drill 3) (layers *.Cu *.Mask))
+    (pad 1 np_thru_hole circle (at -7.5 5 60) (size 3 3) (drill 3) (layers *.Cu *.Mask))
   )
   (module generated:MicroMatch_4p (layer F.Cu)
@@
     (tags "D2PAK D2PAK-3 TO-263AB TO-263")
     (attr smd)
-    (fp_text reference U3 (at 0 -6.3 90) (layer F.SilkS)
+    (fp_text reference U3 (at 11 0) (layer F.SilkS)
       (effects (font (size 1 1) (thickness 0.15)))
     )
@@
       (effects (font (size 1 1) (thickness 0.15)))
     )
+    (fp_line (start 6.95 -5) (end -2.05 -5) (layer F.Fab) (width 0.1))
+    (fp_line (start 6.95 5) (end 6.95 -5) (layer F.Fab) (width 0.1))
+    (fp_line (start -2.05 5) (end 6.95 5) (layer F.Fab) (width 0.1))
+    (fp_line (start -2.05 -5) (end -2.05 5) (layer F.Fab) (width 0.1))
+    (fp_line (start 8.15 -5) (end 6.95 -5) (layer F.Fab) (width 0.1))
+    (fp_line (start 8.15 5) (end 8.15 -5) (layer F.Fab) (width 0.1))
+    (fp_line (start 6.95 5) (end 8.15 5) (layer F.Fab) (width 0.1))
+    (fp_line (start -0.35 -5.1) (end -2.15 -5.1) (layer F.SilkS) (width 0.12))
+    (fp_line (start -2.15 5.1) (end -0.35 5.1) (layer F.SilkS) (width 0.12))
+    (fp_line (start -7.12 -5.65) (end -7.12 5.65) (layer F.CrtYd) (width 0.05))
+    (fp_line (start 9.52 -5.65) (end -7.12 -5.65) (layer F.CrtYd) (width 0.05))
+    (fp_line (start 9.52 -5.65) (end 9.52 5.65) (layer F.CrtYd) (width 0.05))
+    (fp_line (start 9.52 5.65) (end -7.12 5.65) (layer F.CrtYd) (width 0.05))
+    (fp_line (start -2.15 5.1) (end -2.15 4.15) (layer F.SilkS) (width 0.12))
+    (fp_line (start -2.15 -5.1) (end -2.15 -4.15) (layer F.SilkS) (width 0.12))
     (fp_text user %R (at 3.05 0 270) (layer F.Fab)
       (effects (font (size 1 1) (thickness 0.15)))
     )
-    (fp_line (start -2.15 -5.1) (end -2.15 -4.15) (layer F.SilkS) (width 0.12))
-    (fp_line (start -2.15 5.1) (end -2.15 4.15) (layer F.SilkS) (width 0.12))
-    (fp_line (start 9.52 5.65) (end -7.12 5.65) (layer F.CrtYd) (width 0.05))
-    (fp_line (start 9.52 -5.65) (end 9.52 5.65) (layer F.CrtYd) (width 0.05))
-    (fp_line (start 9.52 -5.65) (end -7.12 -5.65) (layer F.CrtYd) (width 0.05))
-    (fp_line (start -7.12 -5.65) (end -7.12 5.65) (layer F.CrtYd) (width 0.05))
-    (fp_line (start -2.15 5.1) (end -0.35 5.1) (layer F.SilkS) (width 0.12))
-    (fp_line (start -0.35 -5.1) (end -2.15 -5.1) (layer F.SilkS) (width 0.12))
-    (fp_line (start 6.95 5) (end 8.15 5) (layer F.Fab) (width 0.1))
-    (fp_line (start 8.15 5) (end 8.15 -5) (layer F.Fab) (width 0.1))
-    (fp_line (start 8.15 -5) (end 6.95 -5) (layer F.Fab) (width 0.1))
-    (fp_line (start -2.05 -5) (end -2.05 5) (layer F.Fab) (width 0.1))
-    (fp_line (start -2.05 5) (end 6.95 5) (layer F.Fab) (width 0.1))
-    (fp_line (start 6.95 5) (end 6.95 -5) (layer F.Fab) (width 0.1))
-    (fp_line (start 6.95 -5) (end -2.05 -5) (layer F.Fab) (width 0.1))
+    (pad 1 smd rect (at -4.58 -3.4 270) (size 4.6 1.1) (layers F.Cu F.Paste F.Mask)
+      (net 18 CTRL2))
+    (pad 3 smd rect (at -4.58 0 270) (size 4.6 1.1) (layers F.Cu F.Paste F.Mask)
+      (net 2 GND))
+    (pad 3 smd rect (at 4.58 0 270) (size 9.4 10.8) (layers F.Cu F.Paste F.Mask)
+      (net 2 GND))
+    (pad 2 smd rect (at -4.58 -1.7 270) (size 4.6 1.1) (layers F.Cu F.Paste F.Mask)
+      (net 1 +5V))
+    (pad 4 smd rect (at -4.58 1.7 270) (size 4.6 1.1) (layers F.Cu F.Paste F.Mask)
+      (net 12 N$4))
     (pad 5 smd rect (at -4.58 3.4 270) (size 4.6 1.1) (layers F.Cu F.Paste F.Mask)
       (net 6 N$3))
-    (pad 4 smd rect (at -4.58 1.7 270) (size 4.6 1.1) (layers F.Cu F.Paste F.Mask)
-      (net 12 N$4))
-    (pad 2 smd rect (at -4.58 -1.7 270) (size 4.6 1.1) (layers F.Cu F.Paste F.Mask)
-      (net 1 +5V))
-    (pad 3 smd rect (at 4.58 0 270) (size 9.4 10.8) (layers F.Cu F.Paste F.Mask)
-      (net 2 GND))
-    (pad 3 smd rect (at -4.58 0 270) (size 4.6 1.1) (layers F.Cu F.Paste F.Mask)
-      (net 2 GND))
-    (pad 1 smd rect (at -4.58 -3.4 270) (size 4.6 1.1) (layers F.Cu F.Paste F.Mask)
-      (net 18 CTRL2))
     (model ${KISYS3DMOD}/TO_SOT_Packages_SMD.3dshapes/TO-263-5Lead.wrl
       (at (xyz -0.18 0 0))
@@
   )
   (module UGL:OSHW_Logo_6mm_height_BCu (layer F.Cu)
-    (at 0 -56)
+    (at 0 -57)
     (descr "OSHW Logo, 6mm height")
     (attr virtual)
@@
       (xy -2.82075 2.070409)) (layer F.Mask) (width 0.01))
   )
+  (gr_text "rev. 1.0\ngithub: wojtekbe/rgbir-lights" (at 0 -51) (layer F.SilkS)
+    (effects (font (size 0.8 0.6) (thickness 0.15)))
+  )
   (gr_line (start 46.24 4.86) (end 41.25 4.86) (layer Edge.Cuts) (width 0.2))
